File: PCB/main/main.kicad_pcb (KiCad board)
At the start: 2 copper layers, 100 x 100 mm, 47 parts, among them J1 Conn_01x33_Female, J2 Conn_01x33_Female, J3 Conn_01x33_Female, J4 Conn_01x33_Female, J5 USB_B_Micro, J6 USB_B_Micro, Q1 2N2222A, SW1 Push Button 1, SW2 C13828, SW3 C13828, U1 TLV316, U2 TP4054

Commit message: Replace main.kicad_pcb
Parts:
- removed BT1: 3V - 4.2V, Battery:BatteryHolder_Keystone_1042_1x18650
- removed C1: 0.33e-6, Capacitor_SMD:C_0201_0603Metric
- removed C2: 1e-6, Capacitor_SMD:C_0201_0603Metric
- removed C3: 0.1e-6, Capacitor_SMD:C_0201_0603Metric
- removed C4: 0.1u, Capacitor_SMD:C_0201_0603Metric
- removed C5: CT41G-0402-2X1-16V-0.1μF-K(N), Capacitor_SMD:C_0201_0603Metric
- removed D1, D2, LED1: 2V, LED_SMD:LED_0805_2012Metric
- removed D3: DIODE, LED_SMD:LED_0805_2012Metric
- removed EEPROM1: AT24C256C-SSHL-T, SOIC127P600X175-8N:EEPROM
- removed FTDI(UART)1: CH340C, CH340C:SOIC127P600X180-16N
- removed J5, J6: USB_B_Micro, Connector_USB:USB_Micro-B_Amphenol_10103594-0001LF_Horizontal
- removed LDR1: 10K - 0.2M, Resistor_SMD:R_0201_0603Metric
- removed LDR2: 10k - 0.2M, Resistor_SMD:R_0201_0603Metric
- removed Q1: 2N2222A, Package_TO_SOT_THT:TO-92
- removed R1: 1650, Resistor_SMD:R_0201_0603Metric
- removed R10, R19, R8: 10K, Resistor_SMD:R_0201_0603Metric
- removed R11, R12, R13, R14: 10k, Resistor_SMD:R_0201_0603Metric
- removed R15, R16, R17, R9: 1K, Resistor_SMD:R_0201_0603Metric
- removed R18: 4K7, Resistor_SMD:R_0201_0603Metric
- removed R2, R6: 100ohms, Resistor_SMD:R_0201_0603Metric
- removed R3: 31ohms, Resistor_SMD:R_0201_0603Metric
- removed R4: 160, Resistor_SMD:R_0201_0603Metric
- removed R5: 10, Resistor_SMD:R_0201_0603Metric
- removed R7: 1000, Resistor_SMD:R_0201_0603Metric
- removed SW1: Push Button 1, 1825910-6:SW_1825910-6-4
- removed SW2, SW3: C13828, 1825910-6:SW_1825910-6-4
- removed TempSensor1: LM75B, LM75BD:SOIC127P600X175-8N
- removed U1: TLV316, Package_TO_SOT_SMD:SOT-23-5
- removed U2: TP4054, Package_TO_SOT_SMD:SOT-23-5
- removed VoltageRegulator1: CJ78M05, Package_TO_SOT_SMD:TO-252-2
Routing:
- net GND: track 421.6 -> 0.00 mm, vias 8 -> 0
- net +5V: track 413.3 -> 0.00 mm, vias 6 -> 0
- net /PA3: track 118.5 -> 0.00 mm, vias 1 -> 0
- net /PA2: track 113.1 -> 0.00 mm, vias 1 -> 0
- net Net-(BT1-Pad1): track 69.0 -> 0.00 mm, vias 2 -> 0
- net Net-(D3-Pad1): track 68.4 -> 0.00 mm, vias 2 -> 0
- net /PC1: track 64.7 -> 0.00 mm, vias 3 -> 0
- net Net-(C5-Pad1): track 64.4 -> 0.00 mm, vias 4 -> 0
- net /PC4: track 56.1 -> 0.00 mm, vias 1 -> 0
- net /microcontroller_interfacing/GND = Normal R/W operations: track 49.6 -> 0.00 mm, vias 2 -> 0
- net Net-(C2-Pad1): track 47.0 -> 0.00 mm
- net USB D-: track 41.0 -> 0.00 mm, vias 2 -> 0
- net /Sensing/I2CBUS: track 35.9 -> 0.00 mm, vias 4 -> 0
- net USB D+: track 35.0 -> 0.00 mm, vias 2 -> 0
- net Net-(Q1-Pad1): track 30.4 -> 0.00 mm, vias 2 -> 0
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Other:
- board outline removed

Commit message: Replace main.kicad_pcb
Parts:
- added BT1: 4.2V-3V, Battery:BatteryHolder_Keystone_1042_1x18650, F.Cu at (140.9, 144.8)
- added C1: 1e-6, Capacitor_SMD:C_0201_0603Metric, F.Cu at (177.1, 83.8)
- added C2: 22u, Capacitor_SMD:C_0805_2012Metric, F.Cu at (198.1, 99.1)
- added C3: 0.1u, Capacitor_SMD:C_0201_0603Metric, F.Cu at (122.5, 100.0)
- added C4: CT41G-0402-2X1-16V-0.1μF-K(N), Capacitor_SMD:C_0201_0603Metric, F.Cu at (114.2, 98.3)
- added D1: 2V, LED_SMD:LED_0805_2012Metric, F.Cu at (176.0, 79.6)
- added D2: 2V, LED_SMD:LED_0805_2012Metric, F.Cu at (203.3, 94.6)
- added D3: 1N5819, Diode_SMD:D_SOD-323, F.Cu at (180.3, 79.6)
- added D4: DIODE, LED_SMD:LED_0805_2012Metric, F.Cu at (112.8, 94.1)
- added EEPROM1: AT24C256C-SSHL-T, SOIC127P600X175-8N:EEPROM, F.Cu at (157.5, 104.1)
- added FTDI(UART)1: CH340C, CH340C:SOIC127P600X180-16N, F.Cu at (111.8, 106.7)
- added J5: USB_B_Micro, Connector_USB:USB_Micro-B_Amphenol_10103594-0001LF_Horizontal, F.Cu at (105.8, 96.5)
- added L1: MLP2012V4R7MT0S1, Inductor_SMD:L_0805_2012Metric, F.Cu at (197.2, 114.3)
- added LDR1: 10K - 0.2M, Resistor_SMD:R_0201_0603Metric, F.Cu at (129.3, 93.5)
- added LDR2: 10k - 0.2M, Resistor_SMD:R_0201_0603Metric, F.Cu at (127.3, 97.0)
- added LED1: 2V, LED_SMD:LED_0805_2012Metric, F.Cu at (123.5, 94.1)
- added Q1: 2N2222A, Package_TO_SOT_THT:TO-92, F.Cu at (164.0, 81.3)
- added R1: 1650, Resistor_SMD:R_0201_0603Metric, F.Cu at (172.2, 83.4)
- added R10: 10k, Resistor_SMD:R_0201_0603Metric, F.Cu at (122.5, 98.3)
- added R11: 10k, Resistor_SMD:R_0201_0603Metric, F.Cu at (127.3, 95.2)
- added R12: 10k, Resistor_SMD:R_0201_0603Metric, F.Cu at (122.5, 96.5)
- added R13: 10k, Resistor_SMD:R_0201_0603Metric, F.Cu at (124.9, 96.5)
- added R14: 10K, Resistor_SMD:R_0201_0603Metric, F.Cu at (111.8, 100.0)
- added R15: 1K, Resistor_SMD:R_0201_0603Metric, F.Cu at (111.8, 96.5)
- added R16: 1K, Resistor_SMD:R_0201_0603Metric, F.Cu at (114.2, 96.5)
- added R17: 1K, Resistor_SMD:R_0201_0603Metric, F.Cu at (116.2, 93.5)
- added R18: 4K7, Resistor_SMD:R_0201_0603Metric, F.Cu at (111.8, 98.3)
- added R2: 100ohms, Resistor_SMD:R_0201_0603Metric, F.Cu at (169.8, 83.4)
- added R3: 100, Resistor_SMD:R_0201_0603Metric, F.Cu at (183.6, 79.0)
- added R4: 100ohms, Resistor_SMD:R_0201_0603Metric, F.Cu at (174.7, 83.8)
- added R5: 1000, Resistor_SMD:R_0201_0603Metric, F.Cu at (197.1, 101.4)
- added R6: 110k, Resistor_SMD:R_0201_0603Metric, F.Cu at (174.9, 82.0)
- added R7: 15k, Resistor_SMD:R_0201_0603Metric, F.Cu at (177.4, 82.0)
- added R8: 10K, Resistor_SMD:R_0201_0603Metric, F.Cu at (124.9, 98.3)
- added R9: 10K, Resistor_SMD:R_0201_0603Metric, F.Cu at (126.9, 93.5)
- added SW1: C13828, 1825910-6:SW_1825910-6-4, F.Cu at (141.4, 111.5)
- added SW2: C13828, 1825910-6:SW_1825910-6-4, F.Cu at (141.4, 104.0)
- added TempSensor1: LM75B, LM75BD:SOIC127P600X175-8N, F.Cu at (111.8, 83.8)
- added U1: TP4054, Package_TO_SOT_SMD:SOT-23-5, F.Cu at (171.1, 80.3)
- added U2: MT3608L, Package_TO_SOT_SMD:SOT-23-6, F.Cu at (198.5, 95.3)
Other:
- board outline added: 100 x 100 mm
