File: PCB/main/main.kicad_pcb (KiCad board)
At the start: 2 copper layers, 100 x 100 mm, 44 parts, among them J1 Conn_01x33_Female, J2 Conn_01x33_Female, J3 Conn_01x33_Female, J4 Conn_01x33_Female, J5 USB_B_Micro, Q1 2N2222A, SW1 C13828, SW2 C13828, U1 TP4054, U2 MT3608L

Commit message: updated microcontroller submodule
Parts:
- added R19: 0, Resistor_SMD:R_0201_0603Metric, F.Cu at (94.0, 99.1)
- added R20: 0, Resistor_SMD:R_0201_0603Metric, F.Cu at (91.5, 99.1)
- moved EEPROM1 22.7 mm to (137.2, 94.0)
Connections:
- net Net-(D4-Pad1) renamed /microcontroller_interfacing/USB Test Point
Changed lines of the file:
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@@
   (net 70 "Net-(D2-Pad2)")
   (net 71 "Net-(D3-Pad2)")
-  (net 72 "Net-(D4-Pad1)")
+  (net 72 "/microcontroller_interfacing/USB Test Point")
   (net 73 "USB D-")
   (net 74 "USB D+")
@@
   (net 92 "unconnected-(FTDI(UART)1-Pad12)")
   (net 93 "unconnected-(FTDI(UART)1-Pad14)")
+  (net 94 "/microcontroller_interfacing/FTDI IN TP")
+  (net 95 "/microcontroller_interfacing/FTDI OUT TP")
   (footprint "Resistor_SMD:R_0201_0603Metric" (layer "F.Cu")
     (at 129.35 93.48)
@@
     )
   )
+  (footprint "Resistor_SMD:R_0201_0603Metric" (layer "F.Cu")
+    (at 93.98 99.06)
+    (descr "Resistor SMD 0201 (0603 Metric), square (rectangular) end terminal, IPC_7351 nominal, (Body size source: https://www.vishay.com/docs/20052/crcw0201e3.pdf), generated with kicad-footprint-generator")
+    (tags "resistor")
+    (property "Sheetfile" "microcontroller_interfacing.kicad_sch")
+    (property "Sheetname" "microcontroller_interfacing")
+    (attr smd)
+    (fp_text reference "R19" (at 0 -1.05) (layer "F.SilkS")
+      (effects (font (size 1 1) (thickness 0.15)))
+    )
+    (fp_text value "0" (at 0 1.05) (layer "F.Fab")
+      (effects (font (size 1 1) (thickness 0.15)))
+    )
+    (fp_text user "${REFERENCE}" (at 0 -0.68) (layer "F.Fab")
+      (effects (font (size 0.25 0.25) (thickness 0.04)))
+    )
+    (fp_line (start -0.7 0.35) (end -0.7 -0.35) (layer "F.CrtYd") (width 0.05))
+    (fp_line (start 0.7 0.35) (end -0.7 0.35) (layer "F.CrtYd") (width 0.05))
+    (fp_line (start -0.7 -0.35) (end 0.7 -0.35) (layer "F.CrtYd") (width 0.05))
+    (fp_line (start 0.7 -0.35) (end 0.7 0.35) (layer "F.CrtYd") (width 0.05))
+    (fp_line (start -0.3 0.15) (end -0.3 -0.15) (layer "F.Fab") (width 0.1))
+    (fp_line (start 0.3 0.15) (end -0.3 0.15) (layer "F.Fab") (width 0.1))
+    (fp_line (start -0.3 -0.15) (end 0.3 -0.15) (layer "F.Fab") (width 0.1))
+    (fp_line (start 0.3 -0.15) (end 0.3 0.15) (layer "F.Fab") (width 0.1))
+    (pad "" smd roundrect (at 0.345 0) (size 0.318 0.36) (layers "F.Paste") (roundrect_rratio 0.25))
+    (pad "" smd roundrect (at -0.345 0) (size 0.318 0.36) (layers "F.Paste") (roundrect_rratio 0.25))
+    (pad "1" smd roundrect (at -0.32 0) (size 0.46 0.4) (layers "F.Cu" "F.Mask") (roundrect_rratio 0.25)
+      (net 54 "/PA9") (pintype "passive"))
+    (pad "2" smd roundrect (at 0.32 0) (size 0.46 0.4) (layers "F.Cu" "F.Mask") (roundrect_rratio 0.25)
+      (net 94 "/microcontroller_interfacing/FTDI IN TP") (pintype "passive"))
+    (model "${KICAD6_3DMODEL_DIR}/Resistor_SMD.3dshapes/R_0201_0603Metric.wrl"
+      (offset (xyz 0 0 0))
+      (scale (xyz 1 1 1))
+      (rotate (xyz 0 0 0))
+    )
+  )
   (footprint "LED_SMD:LED_0805_2012Metric" (layer "F.Cu")
     (at 112.78 94.125)
@@
     (fp_line (start -0.7 -0.6) (end -1 -0.3) (layer "F.Fab") (width 0.1))
     (pad "1" smd roundrect (at -0.9375 0) (size 0.975 1.4) (layers "F.Cu" "F.Paste" "F.Mask") (roundrect_rratio 0.25)
-      (net 72 "Net-(D4-Pad1)") (pinfunction "A") (pintype "passive"))
+      (net 72 "/microcontroller_interfacing/USB Test Point") (pinfunction "A") (pintype "passive"))
     (pad "2" smd roundrect (at 0.9375 0) (size 0.975 1.4) (layers "F.Cu" "F.Paste" "F.Mask") (roundrect_rratio 0.25)
       (net 52 "/PA11") (pinfunction "K") (pintype "passive"))
@@
     )
   )
+  (footprint "Resistor_SMD:R_0201_0603Metric" (layer "F.Cu")
+    (at 91.53 99.06)
+    (descr "Resistor SMD 0201 (0603 Metric), square (rectangular) end terminal, IPC_7351 nominal, (Body size source: https://www.vishay.com/docs/20052/crcw0201e3.pdf), generated with kicad-footprint-generator")
+    (tags "resistor")
+    (property "Sheetfile" "microcontroller_interfacing.kicad_sch")
+    (property "Sheetname" "microcontroller_interfacing")
+    (attr smd)
+    (fp_text reference "R20" (at 0 -1.05) (layer "F.SilkS")
+      (effects (font (size 1 1) (thickness 0.15)))
+    )
+    (fp_text value "0" (at 0 1.05) (layer "F.Fab")
+      (effects (font (size 1 1) (thickness 0.15)))
+    )
+    (fp_text user "${REFERENCE}" (at 0 -0.68) (layer "F.Fab")
+      (effects (font (size 0.25 0.25) (thickness 0.04)))
+    )
+    (fp_line (start 0.7 -0.35) (end 0.7 0.35) (layer "F.CrtYd") (width 0.05))
+    (fp_line (start -0.7 -0.35) (end 0.7 -0.35) (layer "F.CrtYd") (width 0.05))
+    (fp_line (start -0.7 0.35) (end -0.7 -0.35) (layer "F.CrtYd") (width 0.05))
+    (fp_line (start 0.7 0.35) (end -0.7 0.35) (layer "F.CrtYd") (width 0.05))
+    (fp_line (start -0.3 0.15) (end -0.3 -0.15) (layer "F.Fab") (width 0.1))
+    (fp_line (start 0.3 0.15) (end -0.3 0.15) (layer "F.Fab") (width 0.1))
+    (fp_line (start -0.3 -0.15) (end 0.3 -0.15) (layer "F.Fab") (width 0.1))
+    (fp_line (start 0.3 -0.15) (end 0.3 0.15) (layer "F.Fab") (width 0.1))
+    (pad "" smd roundrect (at 0.345 0) (size 0.318 0.36) (layers "F.Paste") (roundrect_rratio 0.25))
+    (pad "" smd roundrect (at -0.345 0) (size 0.318 0.36) (layers "F.Paste") (roundrect_rratio 0.25))
+    (pad "1" smd roundrect (at -0.32 0) (size 0.46 0.4) (layers "F.Cu" "F.Mask") (roundrect_rratio 0.25)
+      (net 53 "/PA10") (pintype "passive"))
+    (pad "2" smd roundrect (at 0.32 0) (size 0.46 0.4) (layers "F.Cu" "F.Mask") (roundrect_rratio 0.25)
+      (net 95 "/microcontroller_interfacing/FTDI OUT TP") (pintype "passive"))
+    (model "${KICAD6_3DMODEL_DIR}/Resistor_SMD.3dshapes/R_0201_0603Metric.wrl"
+      (offset (xyz 0 0 0))
+      (scale (xyz 1 1 1))
+      (rotate (xyz 0 0 0))
+    )
+  )
   (footprint "SOIC127P600X175-8N:EEPROM" (layer "F.Cu")
-    (at 157.48 104.14)
+    (at 137.16 93.98)
     (property "Sheetfile" "microcontroller_interfacing.kicad_sch")
     (property "Sheetname" "microcontroller_interfacing")
@@
     (fp_line (start 3.725 -1.615) (end 3.725 3.335) (layer "F.Fab") (width 0.12))
     (pad "1" smd rect (at -1.325 -1.765 90) (size 1.65 0.4) (layers "F.Cu" "F.Paste" "F.Mask")
-      (net 72 "Net-(D4-Pad1)") (pinfunction "VBUS") (pintype "power_out"))
+      (net 72 "/microcontroller_interfacing/USB Test Point") (pinfunction "VBUS") (pintype "power_out"))
     (pad "2" smd rect (at -0.675 -1.765 90) (size 1.65 0.4) (layers "F.Cu" "F.Paste" "F.Mask")
       (net 73 "USB D-") (pinfunction "D-") (pintype "bidirectional"))

Commit message: updated gerbers and finalized PCB
Parts:
- C4: value CT41G-0402-2X1-16V-0.1μF-K(N) -> 0.1μF
- R1: value 1650 -> 1800
- R3: value 100 -> 100ohms
- R5: value 1000 -> 1200
- moved C2 52.4 mm to (149.9, 78.7)
- moved LDR2 46.9 mm to (162.6, 66.0)
- moved R20 45.9 mm to (136.8, 91.4)
- moved EEPROM1 45.0 mm to (180.3, 81.3), turned to -90 degrees
- moved R19 41.0 mm to (134.3, 91.4)
- moved SW1 40.0 mm to (162.6, 77.6), turned to 180 degrees
- moved R14 36.2 mm to (147.0, 91.4)
- moved L1 34.3 mm to (188.0, 81.3), turned to 180 degrees
- moved R18 33.4 mm to (144.4, 91.4)
- moved R8 33.3 mm to (147.3, 73.7)
- moved FTDI(UART)1 33.1 mm to (129.5, 78.7)
- moved R10 32.2 mm to (142.2, 72.9), turned to 180 degrees
- moved R11 31.8 mm to (144.8, 68.6), turned to 180 degrees
- moved R5 31.0 mm to (190.5, 71.1), turned to -90 degrees
- moved C3 30.8 mm to (144.8, 78.7), turned to 90 degrees
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- renumbered TempSensor1 to TSensor
Connections:
- FTDI(UART)1 pad 15: +5V -> unconnected-(FTDI(UART)1-Pad15)
Routing:
- net /PA8: track 0.00 -> 135.9 mm, vias 0 -> 3
- net Net-(BT1-Pad1): track 0.00 -> 109.0 mm, vias 0 -> 4
- net GND: track 0.00 -> 80.3 mm, vias 0 -> 19
- net /Sensing/I2CBUS: track 0.00 -> 76.2 mm, vias 0 -> 4
- net /Power/Output: track 0.00 -> 75.3 mm, vias 0 -> 2
- net Net-(FTDI(UART)1-Pad13): track 0.00 -> 67.5 mm, vias 0 -> 4
- net /PC1: track 0.00 -> 66.6 mm, vias 0 -> 4
- net Net-(R6-Pad2): track 0.00 -> 66.6 mm, vias 0 -> 3
- net /microcontroller_interfacing/EEPROM MODE TP: track 0.00 -> 56.3 mm, vias 0 -> 2
- net /PC0: track 0.00 -> 50.9 mm
- net /PA9: track 0.00 -> 50.4 mm, vias 0 -> 2
- net /PA10: track 0.00 -> 43.7 mm, vias 0 -> 3
- net USB D+: track 0.00 -> 38.7 mm, vias 0 -> 2
- net /PA11: track 0.00 -> 37.6 mm
- net Net-(D3-Pad2): track 0.00 -> 35.3 mm, vias 0 -> 2
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- added copper zone on F.Cu, net +5V
- added copper zone on B.Cu, net GND
Other:
- board text added: "MT3608L"
- board text added: "t:SW1 b:SW2"
