File: PCB/main/power.kicad_sch (KiCad schematic)
At the start: 17 parts, among them Q1 2N2222A, U1 TP4054, U2 MT3608L

Commit message: Replace power.kicad_sch
Parts:
- C50: renamed from C1; LCSC (none) -> C15849; Price (none) -> 0.0055
- C51: renamed from C2; Extended N -> (none); Populate P -> (none)
- D3: Extended N -> (none); Populate P -> (none)
- D50: renamed from D2; LCSC (none) -> C84256; Price (none) -> 0.0136
- L1: footprint Inductor_SMD:L_0805_2012Metric -> 3088HAT:INDC2012X87N; Extended Y -> (none); Populate P -> (none)
- Q50: renamed from Q1; LCSC (none) -> C118536; Price (none) -> 0.0214
- R50: renamed from R5; value 1000 -> 1200; LCSC (none) -> C22765; Price (none) -> 0.0013
- R51: renamed from R1; value 1650 -> 1800; LCSC (none) -> C4177; Price (none) -> 0.0013
- R52: renamed from R3; value 100 -> 100ohms; LCSC (none) -> C22775; Price (none) -> 0.0012
- R53: renamed from R2; LCSC (none) -> C22775; Price (none) -> 0.0012
- R54: renamed from R4; LCSC (none) -> C22775; Price (none) -> 0.0012
- R55: renamed from R6; Extended N -> (none); Populate P -> (none)
- R56: renamed from R7; Extended N -> (none); Populate P -> (none)
- U1: renamed from U2; Extended Y -> (none)
- U50: renamed from U1; LCSC (none) -> C32574; Price (none) -> 0.1555
- renumbered D1 to D51

Commit message: Replace power.kicad_sch
Parts:
- D51: LCSC (none) -> C84256; Price (none) -> 0..0136
Changed lines of the file:
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@@
+      (effects (font (size 1.27 1.27)) hide)
+    )
+    (property "LCSC" "C84256" (id 4) (at 200.66 88.9 90)
+      (effects (font (size 1.27 1.27)) hide)
+    )
+    (property "Price" "0..0136" (id 5) (at 200.66 88.9 90)
       (effects (font (size 1.27 1.27)) hide)
     )
