File: PCB/main/power.kicad_sch (KiCad schematic)
At the start: 17 parts, among them Q1 2N2222A, U1 TLV316, U2 TP4054

Commit message: new power module
Parts:
- removed C1: 0.33e-6, Capacitor_SMD:C_0201_0603Metric, symbol Device:C
- removed C3: 0.1e-6, Capacitor_SMD:C_0201_0603Metric, symbol Device:C
- removed R4: 160, Resistor_SMD:R_0201_0603Metric, symbol Device:R_Small_US
- removed R5: 10, Resistor_SMD:R_0201_0603Metric, symbol Device:R_Small_US
- removed U1: TLV316, Package_TO_SOT_SMD:SOT-23-5, symbol pspice:OPAMP
- removed VoltageRegulator1: CJ78M05, Package_TO_SOT_SMD:TO-252-2, symbol Regulator_Linear:KA78M05_TO252
- added C51: 22u, Capacitor_SMD:C_0805_2012Metric, symbol Device:C_Small
- added D3: 1N5819, Diode_SMD:D_SOD-323, symbol Diode:1N5819
- added J50: USB_B_Micro, Connector_USB:USB_Micro-B_Amphenol_10103594-0001LF_Horizontal, symbol Connector:USB_B_Micro
- added L1: MLP2012V4R7MT0S1, 3088HAT:INDC2012X87N, symbol Custom:MLP2012V4R7MT0S1
- added R55: 110k, Resistor_SMD:R_0201_0603Metric, symbol Device:R_US
- added R56: 15k, Resistor_SMD:R_0201_0603Metric, symbol Device:R_US
- added U1: MT3608L, Package_TO_SOT_SMD:SOT-23-6, symbol Custom:MT3608L
- BT1: value 3V -> 4.2V-3V
- R52: renamed from R3; value 31ohms -> 100ohms
- renumbered C2 to C50, D2 to D50, D1 to D51, Q1 to Q50, R7 to R50, R1 to R51, R2 to R53, R6 to R54, U2 to U50
Connections:
- net GND: now also C51.2, J50.2 (D-), J50.3 (D+), J50.4 (ID), J50.5 (GND), J50.6 (Shield), R56.2, U1.2 (GND)
- net 5V from USB: no longer names the net of C50.1, R50.2, U50.4 (VDD)
- net 5V from USB: now also J50.1 (VBUS)
- new net: L1.1, U1.4 (EN), U1.5 (Vin)
- new net: D3.2 (A), L1.2, U1.1 (SW)
- new net: R55.2, R56.1, U1.3 (FB)
- new net Output: C51.1, D3.1 (K), R55.1
- no-connect marks 0 -> 1
Other:
- moved on the sheet: D51, Q50, R52, R53, R54

Commit message: Replace power.kicad_sch
Parts:
- removed J50: USB_B_Micro, Connector_USB:USB_Micro-B_Amphenol_10103594-0001LF_Horizontal, symbol Connector:USB_B_Micro
- L1: footprint 3088HAT:INDC2012X87N -> Inductor_SMD:L_0805_2012Metric
- R3: renamed from R52; value 100ohms -> 100
- renumbered C50 to C1, C51 to C2, D51 to D1, D50 to D2, Q50 to Q1, R51 to R1, R53 to R2, R54 to R4, R50 to R5, R55 to R6, R56 to R7, U50 to U1, U1 to U2

Commit message: updated microcontroller submodule
Changed lines of the file:
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@@
     (stroke (width 0) (type default) (color 0 0 0 0))
   )
-  (hierarchical_label "Output" (shape input) (at 254.2794 126.8984 0)
+  (hierarchical_label "Output" (shape output) (at 254.2794 126.8984 0)
     (effects (font (size 1.27 1.27)) (justify left))
   )

Commit message: updated gerbers and finalized PCB
Parts:
- BT1: Populate (none) -> DNP
- C1: LCSC (none) -> C15849; Populate (none) -> P; Price (none) -> 0.0055
- C2, D3, R6, R7: Extended N -> (none)
- D1, D2: LCSC (none) -> C84256; Populate (none) -> P; Price (none) -> 0.0136
- L1: footprint Inductor_SMD:L_0805_2012Metric -> 3088HAT:INDC2012X87N; Extended Y -> (none)
- Q1: LCSC (none) -> C118536; Populate (none) -> P; Price (none) -> 0.0214
- R1: value 1650 -> 1800; LCSC (none) -> C4177; Populate (none) -> P; Price (none) -> 0.0013
- R2, R4: LCSC (none) -> C22775; Populate (none) -> P; Price (none) -> 0.0012
- R3: value 100 -> 100ohms; LCSC (none) -> C22775; Populate (none) -> P; Price (none) -> 0.0012
- R5: value 1000 -> 1200; LCSC (none) -> C22765; Populate (none) -> P; Price (none) -> 0.0013
- U1: LCSC (none) -> C32574; Populate (none) -> P; Price (none) -> 0.1555
- U2: Extended Y -> (none); Populate (none) -> P

Commit message: updated PCB & Assembly file
Parts:
- R2, R3, R4: value 100ohms -> 100
Changed lines of the file:
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@@
       (effects (font (size 1.27 1.27)) (justify left))
     )
-    (property "Value" "100ohms" (id 1) (at 193.04 102.8699 0)
+    (property "Value" "100" (id 1) (at 193.04 102.8699 0)
       (effects (font (size 1.27 1.27)) (justify left))
     )
@@
     (in_bom yes) (on_board yes) (fields_autoplaced)
     (property "Reference" "R4" (id 0) (at 218.44 102.87 90))
-    (property "Value" "100ohms" (id 1) (at 218.44 105.41 90))
+    (property "Value" "100" (id 1) (at 218.44 105.41 90))
     (property "Footprint" "Resistor_SMD:R_0201_0603Metric" (id 2) (at 218.44 109.22 0)
       (effects (font (size 1.27 1.27)) hide)
@@
       (effects (font (size 1.27 1.27)) (justify left))
     )
-    (property "Value" "100ohms" (id 1) (at 203.2 76.1999 0)
-      (effects (font (size 1.27 1.27)) (justify left))
-    )
+    (property "Value" "100" (id 1) (at 203.2 76.1999 0)
+      (effects (font (size 1.27 1.27)) (justify left))
+    )
