File: PCB/main/sensing.kicad_sch (KiCad schematic)
At the start: 13 parts, among them SW1 Push Button 1

Commit message: Replace sensing.kicad_sch
Parts:
- removed R9: 1K, Resistor_SMD:R_0201_0603Metric, symbol Device:R
- removed SW1: Push Button 1, 1825910-6:SW_1825910-6-4, symbol Switch:SW_Push
- renumbered C4 to C3, R11 to R10, R12 to R11, R13 to R12, R14 to R13, R10 to R9
Connections:
- net STM Pin 1 renamed 5V input
Changed lines of the file:
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@@
-    (stroke (width 0) (type default) (color 0 0 0 0))
-  )
-  (wire (pts (xy 139.7 154.94) (xy 147.32 154.94))
-    (stroke (width 0) (type default) (color 0 0 0 0))
-  )
-  (wire (pts (xy 125.73 154.94) (xy 132.08 154.94))
     (stroke (width 0) (type default) (color 0 0 0 0))
   )
@@
   )
   (polyline (pts (xy 97.79 83.82) (xy 97.79 165.1))
-    (stroke (width 0) (type default) (color 0 0 0 0))
-  )
-  (wire (pts (xy 110.49 154.94) (xy 115.57 154.94))
     (stroke (width 0) (type default) (color 0 0 0 0))
   )
@@
     (effects (font (size 1.27 1.27)) (justify left))
   )
-  (hierarchical_label "STM Pin 1" (shape output) (at 245.11 99.06 90)
-    (effects (font (size 1.27 1.27)) (justify left))
-  )
-  (hierarchical_label "STM Pin 1" (shape input) (at 110.49 154.94 180)
-    (effects (font (size 1.27 1.27)) (justify right))
+  (hierarchical_label "5V input" (shape input) (at 245.11 99.06 90)
+    (effects (font (size 1.27 1.27)) (justify left))
   )
   (hierarchical_label "TempSen1" (shape output) (at 255.27 134.62 0)
@@
     (effects (font (size 1.27 1.27)) (justify right))
   )
-  (hierarchical_label "Pushbutton " (shape output) (at 147.32 154.94 0)
-    (effects (font (size 1.27 1.27)) (justify left))
-  )
   (hierarchical_label "LDR1" (shape output) (at 186.69 113.03 0)
     (effects (font (size 1.27 1.27)) (justify left))
@@
     (effects (font (size 1.27 1.27)) (justify right))
   )
-  (hierarchical_label "STM Pin 1" (shape input) (at 121.92 90.17 180)
+  (hierarchical_label "5V input" (shape input) (at 121.92 90.17 180)
     (effects (font (size 1.27 1.27)) (justify right))
   )
@@
     (effects (font (size 1.27 1.27)) (justify left))
   )
-  (hierarchical_label "STM Pin 1" (shape input) (at 271.78 99.06 180)
+  (hierarchical_label "5V input" (shape input) (at 271.78 99.06 180)
     (effects (font (size 1.27 1.27)) (justify right))
   )
   (symbol (lib_id "Device:R") (at 237.49 113.03 0) (unit 1)
     (in_bom yes) (on_board yes) (fields_autoplaced)
-    (property "Reference" "R13" (id 0) (at 240.03 111.7599 0)
+    (property "Reference" "R12" (id 0) (at 240.03 111.7599 0)
       (effects (font (size 1.27 1.27)) (justify left))
     )
@@
   (symbol (lib_id "power:GND") (at 255.27 113.03 0) (unit 1)
     (in_bom yes) (on_board yes) (fields_autoplaced)
-    (property "Reference" "#PWR031" (id 0) (at 255.27 119.38 0)
+    (property "Reference" "#PWR027" (id 0) (at 255.27 119.38 0)
       (effects (font (size 1.27 1.27)) hide)
     )
@@
   (symbol (lib_id "Device:R") (at 147.32 101.6 0) (unit 1)
     (in_bom yes) (on_board yes)
-    (property "Reference" "R10" (id 0) (at 149.86 99.0599 0)
+    (property "Reference" "R9" (id 0) (at 149.86 99.0599 0)
       (effects (font (size 1.27 1.27)) (justify left))
     )
@@
   (symbol (lib_id "Device:R") (at 222.25 113.03 0) (unit 1)
     (in_bom yes) (on_board yes) (fields_autoplaced)
-    (property "Reference" "R11" (id 0) (at 224.79 111.7599 0)
+    (property "Reference" "R10" (id 0) (at 224.79 111.7599 0)
       (effects (font (size 1.27 1.27)) (justify left))
     )
@@
   (symbol (lib_id "power:GND") (at 245.11 149.86 0) (unit 1)
     (in_bom yes) (on_board yes) (fields_autoplaced)
-    (property "Reference" "#PWR030" (id 0) (at 245.11 156.21 0)
+    (property "Reference" "#PWR026" (id 0) (at 245.11 156.21 0)
       (effects (font (size 1.27 1.27)) hide)
     )
@@
   (symbol (lib_id "power:GND") (at 133.35 130.81 0) (unit 1)
     (in_bom yes) (on_board yes) (fields_autoplaced)
-    (property "Reference" "#PWR028" (id 0) (at 133.35 137.16 0)
+    (property "Reference" "#PWR024" (id 0) (at 133.35 137.16 0)
       (effects (font (size 1.27 1.27)) hide)
     )
@@
   (symbol (lib_id "Device:R") (at 271.78 118.11 0) (unit 1)
     (in_bom yes) (on_board yes) (fields_autoplaced)
-    (property "Reference" "R14" (id 0) (at 274.32 116.8399 0)
+    (property "Reference" "R13" (id 0) (at 274.32 116.8399 0)
       (effects (font (size 1.27 1.27)) (justify left))
     )
@@
   (symbol (lib_id "Device:C") (at 255.27 109.22 0) (unit 1)
     (in_bom yes) (on_board yes) (fields_autoplaced)
-    (property "Reference" "C4" (id 0) (at 259.08 107.9499 0)
+    (property "Reference" "C3" (id 0) (at 259.08 107.9499 0)
       (effects (font (size 1.27 1.27)) (justify left))
     )
@@
   (symbol (lib_id "Device:R") (at 229.87 113.03 0) (unit 1)
     (in_bom yes) (on_board yes) (fields_autoplaced)
-    (property "Reference" "R12" (id 0) (at 232.41 111.7599 0)
+    (property "Reference" "R11" (id 0) (at 232.41 111.7599 0)
       (effects (font (size 1.27 1.27)) (justify left))
     )
@@
     (pin "2")
   )
-  (symbol (lib_id "Switch:SW_Push") (at 120.65 154.94 0) (unit 1)
-    (in_bom yes) (on_board yes) (fields_autoplaced)
-    (property "Reference" "SW1" (id 0) (at 120.65 147.32 0))
-    (property "Value" "Push Button 1" (id 1) (at 120.65 149.86 0))
-    (property "Footprint" "1825910-6:SW_1825910-6-4" (id 2) (at 120.65 149.86 0)
-      (effects (font (size 1.27 1.27)) hide)
-    )
-    (property "Datasheet" "~" (id 3) (at 120.65 149.86 0)
-      (effects (font (size 1.27 1.27)) hide)
-    )
-    (pin "1")
-    (pin "2")
-  )
   (symbol (lib_id "power:GND") (at 271.78 143.51 0) (unit 1)
     (in_bom yes) (on_board yes) (fields_autoplaced)
-    (property "Reference" "#PWR032" (id 0) (at 271.78 149.86 0)
+    (property "Reference" "#PWR028" (id 0) (at 271.78 149.86 0)
       (effects (font (size 1.27 1.27)) hide)
     )
@@
   (symbol (lib_id "power:GND") (at 147.32 139.7 0) (unit 1)
     (in_bom yes) (on_board yes) (fields_autoplaced)
-    (property "Reference" "#PWR029" (id 0) (at 147.32 146.05 0)
+    (property "Reference" "#PWR025" (id 0) (at 147.32 146.05 0)
       (effects (font (size 1.27 1.27)) hide)
     )
@@
       (effects (font (size 1.27 1.27)) hide)
     )
-    (pin "1")
-    (pin "2")
-  )
-  (symbol (lib_id "Device:R") (at 135.89 154.94 270) (unit 1)
-    (in_bom yes) (on_board yes)
-    (property "Reference" "R9" (id 0) (at 137.16 149.86 90))
-    (property "Value" "1K" (id 1) (at 137.16 152.4 90))
-    (property "Footprint" "Resistor_SMD:R_0201_0603Metric" (id 2) (at 142.24 158.75 90)
-      (effects (font (size 1.27 1.27)) hide)
-    )
-    (property "Datasheet" "~" (id 3) (at 135.89 154.94 0)
-      (effects (font (size 1.27 1.27)) hide)
-    )

Commit message: Replace sensing.kicad_sch
Parts:
- C1: renamed from C3; LCSC (none) -> C141382; Price (none) -> 0.0032
- LDR1, LDR2: LCSC (none) -> C779572; Price (none) -> 0.0503
- LED1: LCSC (none) -> C84256; Price (none) -> 0.0136
- R1: renamed from R8; LCSC (none) -> C25804; Price (none) -> 0.0012
- R2: renamed from R9; LCSC (none) -> C25804; Price (none) -> 0.0012
- R4: renamed from R10; LCSC (none) -> C25804; Price (none) -> 0.0012
- R5: renamed from R11; LCSC (none) -> C25804; Price (none) -> 0.0012
- R6: renamed from R12; LCSC (none) -> C25804; Price (none) -> 0.0012
- R7: renamed from R13; LCSC (none) -> C25804; Price (none) -> 0.0012
- TempSensor1: LCSC (none) -> C2837470; Price (none) -> 0.4002
Changed lines of the file:
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@@
   (symbol (lib_id "Device:R") (at 237.49 113.03 0) (unit 1)
     (in_bom yes) (on_board yes) (fields_autoplaced)
-    (property "Reference" "R12" (id 0) (at 240.03 111.7599 0)
+    (property "Reference" "R6" (id 0) (at 240.03 111.7599 0)
       (effects (font (size 1.27 1.27)) (justify left))
     )
@@
       (effects (font (size 1.27 1.27)) hide)
     )
+    (property "LCSC" "C25804" (id 4) (at 237.49 113.03 0)
+      (effects (font (size 1.27 1.27)) hide)
+    )
+    (property "Price" "0.0012" (id 5) (at 237.49 113.03 0)
+      (effects (font (size 1.27 1.27)) hide)
+    )
     (pin "1")
     (pin "2")
@@
   (symbol (lib_id "power:GND") (at 255.27 113.03 0) (unit 1)
     (in_bom yes) (on_board yes) (fields_autoplaced)
-    (property "Reference" "#PWR027" (id 0) (at 255.27 119.38 0)
+    (property "Reference" "#PWR0101" (id 0) (at 255.27 119.38 0)
       (effects (font (size 1.27 1.27)) hide)
     )
@@
   (symbol (lib_id "Device:R") (at 147.32 101.6 0) (unit 1)
     (in_bom yes) (on_board yes)
-    (property "Reference" "R9" (id 0) (at 149.86 99.0599 0)
+    (property "Reference" "R2" (id 0) (at 149.86 99.0599 0)
       (effects (font (size 1.27 1.27)) (justify left))
     )
@@
       (effects (font (size 1.27 1.27)) hide)
     )
+    (property "LCSC" "C25804" (id 4) (at 147.32 101.6 0)
+      (effects (font (size 1.27 1.27)) hide)
+    )
+    (property "Price" "0.0012" (id 5) (at 147.32 101.6 0)
+      (effects (font (size 1.27 1.27)) hide)
+    )
     (pin "1")
     (pin "2")
@@
       (effects (font (size 1.27 1.27)) hide)
     )
+    (property "LCSC" "C84256" (id 4) (at 271.78 132.08 90)
+      (effects (font (size 1.27 1.27)) hide)
+    )
+    (property "Price" "0.0136" (id 5) (at 271.78 132.08 90)
+      (effects (font (size 1.27 1.27)) hide)
+    )
     (pin "1")
     (pin "2")
@@
   (symbol (lib_id "Device:R") (at 222.25 113.03 0) (unit 1)
     (in_bom yes) (on_board yes) (fields_autoplaced)
-    (property "Reference" "R10" (id 0) (at 224.79 111.7599 0)
+    (property "Reference" "R4" (id 0) (at 224.79 111.7599 0)
       (effects (font (size 1.27 1.27)) (justify left))
     )
@@
       (effects (font (size 1.27 1.27)) hide)
     )
+    (property "LCSC" "C25804" (id 4) (at 222.25 113.03 0)
+      (effects (font (size 1.27 1.27)) hide)
+    )
+    (property "Price" "0.0012" (id 5) (at 222.25 113.03 0)
+      (effects (font (size 1.27 1.27)) hide)
+    )
     (pin "1")
     (pin "2")
@@
   (symbol (lib_id "power:GND") (at 245.11 149.86 0) (unit 1)
     (in_bom yes) (on_board yes) (fields_autoplaced)
-    (property "Reference" "#PWR026" (id 0) (at 245.11 156.21 0)
+    (property "Reference" "#PWR0103" (id 0) (at 245.11 156.21 0)
       (effects (font (size 1.27 1.27)) hide)
     )
@@
   (symbol (lib_id "power:GND") (at 133.35 130.81 0) (unit 1)
     (in_bom yes) (on_board yes) (fields_autoplaced)
-    (property "Reference" "#PWR024" (id 0) (at 133.35 137.16 0)
+    (property "Reference" "#PWR0104" (id 0) (at 133.35 137.16 0)
       (effects (font (size 1.27 1.27)) hide)
     )
@@
   (symbol (lib_id "Device:R") (at 271.78 118.11 0) (unit 1)
     (in_bom yes) (on_board yes) (fields_autoplaced)
-    (property "Reference" "R13" (id 0) (at 274.32 116.8399 0)
+    (property "Reference" "R7" (id 0) (at 274.32 116.8399 0)
       (effects (font (size 1.27 1.27)) (justify left))
     )
@@
     )
     (property "Datasheet" "~" (id 3) (at 271.78 118.11 0)
+      (effects (font (size 1.27 1.27)) hide)
+    )
+    (property "LCSC" "C25804" (id 4) (at 271.78 118.11 0)
+      (effects (font (size 1.27 1.27)) hide)
+    )
+    (property "Price" "0.0012" (id 5) (at 271.78 118.11 0)
       (effects (font (size 1.27 1.27)) hide)
     )
@@
       (effects (font (size 1.27 1.27)) hide)
     )
+    (property "LCSC" "C779572" (id 4) (at 133.35 119.38 0)
+      (effects (font (size 1.27 1.27)) hide)
+    )
+    (property "Price" "0.0503" (id 5) (at 133.35 119.38 0)
+      (effects (font (size 1.27 1.27)) hide)
+    )
     (pin "1")
     (pin "2")
@@
   (symbol (lib_id "Device:C") (at 255.27 109.22 0) (unit 1)
     (in_bom yes) (on_board yes) (fields_autoplaced)
-    (property "Reference" "C3" (id 0) (at 259.08 107.9499 0)
+    (property "Reference" "C1" (id 0) (at 259.08 107.9499 0)
       (effects (font (size 1.27 1.27)) (justify left))
     )
@@
     )
     (property "Datasheet" "~" (id 3) (at 255.27 109.22 0)
+      (effects (font (size 1.27 1.27)) hide)
+    )
+    (property "LCSC" "C141382" (id 4) (at 255.27 109.22 0)
+      (effects (font (size 1.27 1.27)) hide)
+    )
+    (property "Price" "0.0032" (id 5) (at 255.27 109.22 0)
       (effects (font (size 1.27 1.27)) hide)
     )
@@
   (symbol (lib_id "Device:R") (at 133.35 101.6 0) (unit 1)
     (in_bom yes) (on_board yes)
-    (property "Reference" "R8" (id 0) (at 135.89 99.0599 0)
+    (property "Reference" "R1" (id 0) (at 135.89 99.0599 0)
       (effects (font (size 1.27 1.27)) (justify left))
     )
@@
       (effects (font (size 1.27 1.27)) hide)
     )
+    (property "LCSC" "C25804" (id 4) (at 133.35 101.6 0)
+      (effects (font (size 1.27 1.27)) hide)
+    )
+    (property "Price" "0.0012" (id 5) (at 133.35 101.6 0)
+      (effects (font (size 1.27 1.27)) hide)
+    )
     (pin "1")
     (pin "2")
@@
   (symbol (lib_id "Device:R") (at 229.87 113.03 0) (unit 1)
     (in_bom yes) (on_board yes) (fields_autoplaced)
-    (property "Reference" "R11" (id 0) (at 232.41 111.7599 0)
+    (property "Reference" "R5" (id 0) (at 232.41 111.7599 0)
       (effects (font (size 1.27 1.27)) (justify left))
     )
@@
       (effects (font (size 1.27 1.27)) hide)
     )
+    (property "LCSC" "C25804" (id 4) (at 229.87 113.03 0)
+      (effects (font (size 1.27 1.27)) hide)
+    )
+    (property "Price" "0.0012" (id 5) (at 229.87 113.03 0)
+      (effects (font (size 1.27 1.27)) hide)
+    )
     (pin "1")
     (pin "2")
@@
   (symbol (lib_id "power:GND") (at 271.78 143.51 0) (unit 1)
     (in_bom yes) (on_board yes) (fields_autoplaced)
-    (property "Reference" "#PWR028" (id 0) (at 271.78 149.86 0)
+    (property "Reference" "#PWR0102" (id 0) (at 271.78 149.86 0)
       (effects (font (size 1.27 1.27)) hide)
     )
@@
     )
     (property "Datasheet" "http://www.ti.com/lit/ds/symlink/lm75b.pdf" (id 3) (at 245.11 137.16 0)
+      (effects (font (size 1.27 1.27)) hide)
+    )
+    (property "LCSC" "C2837470" (id 4) (at 245.11 137.16 0)
+      (effects (font (size 1.27 1.27)) hide)
+    )
+    (property "Price" "0.4002" (id 5) (at 245.11 137.16 0)
       (effects (font (size 1.27 1.27)) hide)
     )
@@
   (symbol (lib_id "power:GND") (at 147.32 139.7 0) (unit 1)
     (in_bom yes) (on_board yes) (fields_autoplaced)
-    (property "Reference" "#PWR025" (id 0) (at 147.32 146.05 0)
+    (property "Reference" "#PWR0105" (id 0) (at 147.32 146.05 0)
       (effects (font (size 1.27 1.27)) hide)
     )
@@
     )
     (property "Datasheet" "~" (id 3) (at 147.32 132.08 0)
+      (effects (font (size 1.27 1.27)) hide)
+    )
+    (property "LCSC" "C779572" (id 4) (at 147.32 130.81 0)
+      (effects (font (size 1.27 1.27)) hide)
+    )
+    (property "Price" "0.0503" (id 5) (at 147.32 130.81 0)
       (effects (font (size 1.27 1.27)) hide)
     )
@@
       (reference "R2") (unit 1) (value "10K") (footprint "Resistor_SMD:R_0201_0603Metric")
     )
-    (path "/fee6e0a9-3581-4681-828a-d7e7c0b72a48"
-      (reference "R3") (unit 1) (value "1K") (footprint "Resistor_SMD:R_0201_0603Metric")
-    )
     (path "/3d24ca64-8898-4a21-92dc-4bb372c9b113"
       (reference "R4") (unit 1) (value "10k") (footprint "Resistor_SMD:R_0201_0603Metric")
@@
       (reference "R7") (unit 1) (value "10k") (footprint "Resistor_SMD:R_0201_0603Metric")
     )
-    (path "/b35b18ad-0223-451a-bb16-91d2a55a057e"
-      (reference "SW1") (unit 1) (value "Push Button 1") (footprint "")
-    )
     (path "/ee0404f1-775a-4f9c-8b75-b98271704a27"
-      (reference "TempSensor1") (unit 1) (value "LM75B") (footprint "")
-    )
-  )
+      (reference "TempSensor1") (unit 1) (value "LM75B") (footprint "LM75BD:SOIC127P600X175-8N")
+    )
+  )
