File: PCB/main/sensing.kicad_sch (KiCad schematic)
At the start: 11 parts

Commit message: added new jlcpcb files. other group members to double check
Parts:
- TempSensor1: Alt_LCSC (none) -> C2837470
Changed lines of the file:
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@@
+      (effects (font (size 1.27 1.27)) hide)
+    )
+    (property "Alt_LCSC" "C2837470" (id 7) (at 245.11 137.16 0)
       (effects (font (size 1.27 1.27)) hide)
     )

Commit message: updated PCB & Assembly file
Parts:
- TempSensor1: footprint LM75BD:SOIC127P600X175-8N -> Package_SO:MSOP-8_3x3mm_P0.65mm
Changed lines of the file:
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@@
       (effects (font (size 1.27 1.27)) (justify left))
     )
-    (property "Footprint" "LM75BD:SOIC127P600X175-8N" (id 2) (at 245.11 137.16 0)
+    (property "Footprint" "Package_SO:MSOP-8_3x3mm_P0.65mm" (id 2) (at 245.11 137.16 0)
       (effects (font (size 1.27 1.27)) hide)
     )
